File: kicad/_autosave-Super7Seg.kicad_pcb (KiCad board)
At the start: 2 copper layers, 40 parts, among them CON1 AVR-ISP-6, IC1 ATMEGA328P-P, P1 UART, P2 CONN_01X02, P3 CONN_01X02, Q1 PN2222ABU, Q2 PN2907BU, Q3 PN2222ABU, Q4 PN2907BU, Q5 PN2222ABU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

Commit message: still trying to get the layout
Parts:
- added REF**: TQFP-32_7x7mm_Pitch0.8mm, Housings_QFP:TQFP-32_7x7mm_Pitch0.8mm, F.Cu at (154.3, 79.4)
