File: kicad/_saved_Super7Seg.sch (KiCad schematic (older format))
At the start: 44 parts, among them CON1 AVR-ISP-6, IC1 ATMEGA328P-P, P1 CONN_01X13, P1 UART, P2 CONN_01X02, P2 CONN_01X09, P3 CONN_01X02, P3 CONN_01X13, P4 CONN_01X09

Commit message: new layout plan
Parts:
- P1, P3: footprint (none) -> Socket_Strips:Socket_Strip_Straight_1x13
- P2, P4: footprint (none) -> Socket_Strips:Socket_Strip_Straight_1x09
- renumbered P1 to P5, P2 to P6, P3 to P7
Changed lines of the file:
@@
 	7450 1200 7500 1200
 $Comp
-L CONN_01X06 P1
+L CONN_01X06 P5
 U 1 1 585E6DD7
 P 6050 1150
-F 0 "P1" H 6050 1500 50  0000 C CNN
+F 0 "P5" H 6050 1500 50  0000 C CNN
 F 1 "UART" V 6150 1150 50  0000 C CNN
 F 2 "Socket_Strips:Socket_Strip_Straight_1x06" H 6050 1150 50  0001 C CNN
@@
 $EndComp
 $Comp
-L PWR_FLAG #FLG010
+L PWR_FLAG #FLG07
 U 1 1 585EE745
 P 5600 3800
-F 0 "#FLG010" H 5600 3895 50  0001 C CNN
+F 0 "#FLG07" H 5600 3895 50  0001 C CNN
 F 1 "PWR_FLAG" H 5600 3980 50  0000 C CNN
 F 2 "" H 5600 3800 50  0000 C CNN
@@
 $EndComp
 $Comp
-L GND #PWR011
+L GND #PWR08
 U 1 1 585EEC8B
 P 5600 3850
-F 0 "#PWR011" H 5600 3600 50  0001 C CNN
+F 0 "#PWR08" H 5600 3600 50  0001 C CNN
 F 1 "GND" H 5600 3700 50  0000 C CNN
 F 2 "" H 5600 3850 50  0000 C CNN
@@
 $EndComp
 $Comp
-L VCC #PWR012
+L VCC #PWR09
 U 1 1 585EED05
 P 6050 3850
-F 0 "#PWR012" H 6050 3700 50  0001 C CNN
+F 0 "#PWR09" H 6050 3700 50  0001 C CNN
 F 1 "VCC" H 6050 4000 50  0000 C CNN
 F 2 "" H 6050 3850 50  0000 C CNN
@@
 $EndComp
 $Comp
-L PWR_FLAG #FLG013
+L PWR_FLAG #FLG010
 U 1 1 585EED7F
 P 6050 3800
-F 0 "#FLG013" H 6050 3895 50  0001 C CNN
+F 0 "#FLG010" H 6050 3895 50  0001 C CNN
 F 1 "PWR_FLAG" H 6050 3980 50  0000 C CNN
 F 2 "" H 6050 3800 50  0000 C CNN
@@
 	6750 4100 6750 4000
 $Comp
-L VCC #PWR014
+L VCC #PWR011
 U 1 1 585F09FF
 P 5850 1100
-F 0 "#PWR014" H 5850 950 50  0001 C CNN
+F 0 "#PWR011" H 5850 950 50  0001 C CNN
 F 1 "VCC" V 5850 1300 50  0000 C CNN
 F 2 "" H 5850 1100 50  0000 C CNN
@@
 $EndComp
 $Comp
-L GND #PWR015
+L GND #PWR012
 U 1 1 585F0B43
 P 5850 900
-F 0 "#PWR015" H 5850 650 50  0001 C CNN
+F 0 "#PWR012" H 5850 650 50  0001 C CNN
 F 1 "GND" V 5850 700 50  0000 C CNN
 F 2 "" H 5850 900 50  0000 C CNN
@@
 $EndComp
 $Comp
-L CONN_01X02 P2
+L CONN_01X02 P6
 U 1 1 585F7453
 P 6050 1850
-F 0 "P2" H 6050 2000 50  0000 C CNN
+F 0 "P6" H 6050 2000 50  0000 C CNN
 F 1 "CONN_01X02" V 6150 1850 50  0000 C CNN
 F 2 "Socket_Strips:Socket_Strip_Straight_1x02" H 6050 1850 50  0001 C CNN
@@
 $EndComp
 $Comp
-L GND #PWR016
+L GND #PWR013
 U 1 1 585F7588
 P 5850 1800
-F 0 "#PWR016" H 5850 1550 50  0001 C CNN
+F 0 "#PWR013" H 5850 1550 50  0001 C CNN
 F 1 "GND" V 5850 1600 50  0000 C CNN
 F 2 "" H 5850 1800 50  0000 C CNN
@@
 RX
 $Comp
-L CONN_01X02 P3
+L CONN_01X02 P7
 U 1 1 585F771C
 P 6050 2400
-F 0 "P3" H 6050 2550 50  0000 C CNN
+F 0 "P7" H 6050 2550 50  0000 C CNN
 F 1 "CONN_01X02" V 6150 2400 50  0000 C CNN
 F 2 "Socket_Strips:Socket_Strip_Straight_1x02" H 6050 2400 50  0001 C CNN
@@
 $EndComp
 $Comp
-L GND #PWR017
+L GND #PWR014
 U 1 1 585F7722
 P 5850 2350
-F 0 "#PWR017" H 5850 2100 50  0001 C CNN
+F 0 "#PWR014" H 5850 2100 50  0001 C CNN
 F 1 "GND" V 5850 2150 50  0000 C CNN
 F 2 "" H 5850 2350 50  0000 C CNN
@@
 TX
 $Comp
-L GND #PWR018
+L GND #PWR015
 U 1 1 585F7F59
 P 7400 4950
-F 0 "#PWR018" H 7400 4700 50  0001 C CNN
+F 0 "#PWR015" H 7400 4700 50  0001 C CNN
 F 1 "GND" V 7400 4750 50  0000 C CNN
 F 2 "" H 7400 4950 50  0000 C CNN
@@
 MISO
 $Comp
-L VCC #PWR019
+L VCC #PWR016
 U 1 1 585F951B
 P 7400 4750
-F 0 "#PWR019" H 7400 4600 50  0001 C CNN
+F 0 "#PWR016" H 7400 4600 50  0001 C CNN
 F 1 "VCC" H 7400 4900 50  0000 C CNN
 F 2 "" H 7400 4750 50  0000 C CNN
@@
 Connection ~ 11100 3450
 $Comp
-L GND #PWR?
+L GND #PWR017
 U 1 1 5866B73D
 P 11500 3750
-F 0 "#PWR?" H 11500 3500 50  0001 C CNN
+F 0 "#PWR017" H 11500 3500 50  0001 C CNN
 F 1 "GND" H 11500 3600 50  0000 C CNN
 F 2 "" H 11500 3750 50  0000 C CNN
@@
 Connection ~ 11100 4000
 $Comp
-L GND #PWR?
+L GND #PWR018
 U 1 1 58670988
 P 11500 4300
-F 0 "#PWR?" H 11500 4050 50  0001 C CNN
+F 0 "#PWR018" H 11500 4050 50  0001 C CNN
 F 1 "GND" H 11500 4150 50  0000 C CNN
 F 2 "" H 11500 4300 50  0000 C CNN
@@
 Connection ~ 11100 4550
 $Comp
-L GND #PWR?
+L GND #PWR019
 U 1 1 58670A45
 P 11500 4850
-F 0 "#PWR?" H 11500 4600 50  0001 C CNN
+F 0 "#PWR019" H 11500 4600 50  0001 C CNN
 F 1 "GND" H 11500 4700 50  0000 C CNN
 F 2 "" H 11500 4850 50  0000 C CNN
@@
 F 0 "P3" H 10850 3050 50  0000 C CNN
 F 1 "CONN_01X13" V 10950 2350 50  0000 C CNN
-F 2 "" H 10850 2350 50  0000 C CNN
+F 2 "Socket_Strips:Socket_Strip_Straight_1x13" H 10850 2350 50  0001 C CNN
 F 3 "" H 10850 2350 50  0000 C CNN
 	1    10850 2350
@@
 F 0 "P4" H 10850 3150 50  0000 C CNN
 F 1 "CONN_01X09" V 10950 2650 50  0000 C CNN
-F 2 "" H 10850 2650 50  0000 C CNN
+F 2 "Socket_Strips:Socket_Strip_Straight_1x09" H 10850 2650 50  0001 C CNN
 F 3 "" H 10850 2650 50  0000 C CNN
 	1    10850 2650
@@
 F 0 "P1" H 3050 6900 50  0000 C CNN
 F 1 "CONN_01X13" V 3150 6200 50  0000 C CNN
-F 2 "" H 3050 6200 50  0000 C CNN
+F 2 "Socket_Strips:Socket_Strip_Straight_1x13" H 3050 6200 50  0001 C CNN
 F 3 "" H 3050 6200 50  0000 C CNN
 	1    3050 6200
@@
 F 0 "P2" H 3050 7000 50  0000 C CNN
 F 1 "CONN_01X09" V 3150 6500 50  0000 C CNN
-F 2 "" H 3050 6500 50  0000 C CNN
+F 2 "Socket_Strips:Socket_Strip_Straight_1x09" H 3050 6500 50  0001 C CNN
 F 3 "" H 3050 6500 50  0000 C CNN
 	1    3050 6500
