File: kicad/_saved_Super7Seg.sch (KiCad schematic (older format))
At the start: 36 parts, among them CON1 AVR-ISP-6, IC1 ATMEGA328P-P, IC2 74HC238, P1 CONN_01X13, P2 CONN_01X09, P3 CONN_01X13, P4 CONN_01X09, P5 UART, P6 CONN_01X02, P7 CONN_01X02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

Commit message: Removed AREF cap.
Parts:
- IC2, U1: footprint (none) -> Housings_DIP:DIP-16_W7.62mm
- P5: footprint Socket_Strips:Socket_Strip_Straight_1x06 -> misc:Strip_1x06
- P6, P7: footprint Socket_Strips:Socket_Strip_Straight_1x02 -> misc:Strip_1x02
- renumbered C2 to C1, C3 to C2
Changed lines of the file:
@@
 	6750 1650 6750 2400
 $Comp
-L C_Small C2
+L C_Small C1
 U 1 1 585DF6FF
 P 6700 3150
-F 0 "C2" H 6710 3220 50  0000 L CNN
+F 0 "C1" H 6710 3220 50  0000 L CNN
 F 1 "0.1uF" H 6710 3070 50  0000 L CNN
 F 2 "Capacitors_ThroughHole:C_Disc_D3_P2.5" H 6700 3150 50  0001 C CNN
@@
 RESET
 $Comp
-L C_Small C3
+L C_Small C2
 U 1 1 585E2D7F
 P 7600 1200
-F 0 "C3" H 7610 1270 50  0000 L CNN
+F 0 "C2" H 7610 1270 50  0000 L CNN
 F 1 "0.1uF" H 7610 1120 50  0000 L CNN
 F 2 "Capacitors_ThroughHole:C_Disc_D3_P2.5" H 7600 1200 50  0001 C CNN
@@
 F 0 "P5" H 6050 1500 50  0000 C CNN
 F 1 "UART" V 6150 1150 50  0000 C CNN
-F 2 "Socket_Strips:Socket_Strip_Straight_1x06" H 6050 1150 50  0001 C CNN
+F 2 "misc:Strip_1x06" H 6050 1150 50  0001 C CNN
 F 3 "" H 6050 1150 50  0000 C CNN
 	1    6050 1150
@@
 $EndComp
 $Comp
-L PWR_FLAG #FLG07
+L PWR_FLAG #FLG06
 U 1 1 585EE745
 P 5600 3800
-F 0 "#FLG07" H 5600 3895 50  0001 C CNN
+F 0 "#FLG06" H 5600 3895 50  0001 C CNN
 F 1 "PWR_FLAG" H 5600 3980 50  0000 C CNN
 F 2 "" H 5600 3800 50  0000 C CNN
@@
 $EndComp
 $Comp
-L GND #PWR08
+L GND #PWR07
 U 1 1 585EEC8B
 P 5600 3850
-F 0 "#PWR08" H 5600 3600 50  0001 C CNN
+F 0 "#PWR07" H 5600 3600 50  0001 C CNN
 F 1 "GND" H 5600 3700 50  0000 C CNN
 F 2 "" H 5600 3850 50  0000 C CNN
@@
 $EndComp
 $Comp
-L VCC #PWR09
+L VCC #PWR08
 U 1 1 585EED05
 P 6050 3850
-F 0 "#PWR09" H 6050 3700 50  0001 C CNN
+F 0 "#PWR08" H 6050 3700 50  0001 C CNN
 F 1 "VCC" H 6050 4000 50  0000 C CNN
 F 2 "" H 6050 3850 50  0000 C CNN
@@
 $EndComp
 $Comp
-L PWR_FLAG #FLG010
+L PWR_FLAG #FLG09
 U 1 1 585EED7F
 P 6050 3800
-F 0 "#FLG010" H 6050 3895 50  0001 C CNN
+F 0 "#FLG09" H 6050 3895 50  0001 C CNN
 F 1 "PWR_FLAG" H 6050 3980 50  0000 C CNN
 F 2 "" H 6050 3800 50  0000 C CNN
@@
 	6750 4100 6750 4000
 $Comp
-L VCC #PWR011
+L VCC #PWR010
 U 1 1 585F09FF
 P 5850 1100
-F 0 "#PWR011" H 5850 950 50  0001 C CNN
+F 0 "#PWR010" H 5850 950 50  0001 C CNN
 F 1 "VCC" V 5850 1300 50  0000 C CNN
 F 2 "" H 5850 1100 50  0000 C CNN
@@
 $EndComp
 $Comp
-L GND #PWR012
+L GND #PWR011
 U 1 1 585F0B43
 P 5850 900
-F 0 "#PWR012" H 5850 650 50  0001 C CNN
+F 0 "#PWR011" H 5850 650 50  0001 C CNN
 F 1 "GND" V 5850 700 50  0000 C CNN
 F 2 "" H 5850 900 50  0000 C CNN
@@
 F 0 "P6" H 6050 2000 50  0000 C CNN
 F 1 "CONN_01X02" V 6150 1850 50  0000 C CNN
-F 2 "Socket_Strips:Socket_Strip_Straight_1x02" H 6050 1850 50  0001 C CNN
+F 2 "misc:Strip_1x02" H 6050 1850 50  0001 C CNN
 F 3 "" H 6050 1850 50  0000 C CNN
 	1    6050 1850
@@
 $EndComp
 $Comp
-L GND #PWR013
+L GND #PWR012
 U 1 1 585F7588
 P 5850 1800
-F 0 "#PWR013" H 5850 1550 50  0001 C CNN
+F 0 "#PWR012" H 5850 1550 50  0001 C CNN
 F 1 "GND" V 5850 1600 50  0000 C CNN
 F 2 "" H 5850 1800 50  0000 C CNN
@@
 F 0 "P7" H 6050 2550 50  0000 C CNN
 F 1 "CONN_01X02" V 6150 2400 50  0000 C CNN
-F 2 "Socket_Strips:Socket_Strip_Straight_1x02" H 6050 2400 50  0001 C CNN
+F 2 "misc:Strip_1x02" H 6050 2400 50  0001 C CNN
 F 3 "" H 6050 2400 50  0000 C CNN
 	1    6050 2400
@@
 $EndComp
 $Comp
-L GND #PWR014
+L GND #PWR013
 U 1 1 585F7722
 P 5850 2350
-F 0 "#PWR014" H 5850 2100 50  0001 C CNN
+F 0 "#PWR013" H 5850 2100 50  0001 C CNN
 F 1 "GND" V 5850 2150 50  0000 C CNN
 F 2 "" H 5850 2350 50  0000 C CNN
@@
 TX
 $Comp
-L GND #PWR015
+L GND #PWR014
 U 1 1 585F7F59
 P 7400 4950
-F 0 "#PWR015" H 7400 4700 50  0001 C CNN
+F 0 "#PWR014" H 7400 4700 50  0001 C CNN
 F 1 "GND" V 7400 4750 50  0000 C CNN
 F 2 "" H 7400 4950 50  0000 C CNN
@@
 MISO
 $Comp
-L VCC #PWR016
+L VCC #PWR015
 U 1 1 585F951B
 P 7400 4750
-F 0 "#PWR016" H 7400 4600 50  0001 C CNN
+F 0 "#PWR015" H 7400 4600 50  0001 C CNN
 F 1 "VCC" H 7400 4900 50  0000 C CNN
 F 2 "" H 7400 4750 50  0000 C CNN
@@
 F 0 "U1" H 12100 4150 50  0000 C CNN
 F 1 "ULN2003A" H 12100 3950 50  0000 C CNN
-F 2 "" H 12100 4050 50  0000 C CNN
+F 2 "Housings_DIP:DIP-16_W7.62mm" H 12100 4050 50  0001 C CNN
 F 3 "" H 12100 4050 50  0000 C CNN
 	1    12100 4050
@@
 F 0 "IC2" H 10800 4650 60  0000 C CNN
 F 1 "74HC238" H 10950 3350 60  0000 C CNN
-F 2 "" H 10950 4000 60  0000 C CNN
+F 2 "Housings_DIP:DIP-16_W7.62mm" H 10950 4000 60  0001 C CNN
 F 3 "" H 10950 4000 60  0000 C CNN
 	1    10950 4000
@@
 $EndComp
 $Comp
-L GND #PWR?
+L GND #PWR016
 U 1 1 586ACCF7
 P 10500 4300
-F 0 "#PWR?" H 10500 4050 50  0001 C CNN
+F 0 "#PWR016" H 10500 4050 50  0001 C CNN
 F 1 "GND" H 10500 4150 50  0000 C CNN
 F 2 "" H 10500 4300 50  0000 C CNN
@@
 	10550 4300 10550 4400
 $Comp
-L VCC #PWR?
+L VCC #PWR017
 U 1 1 586ADBCB
 P 10500 4500
-F 0 "#PWR?" H 10500 4350 50  0001 C CNN
+F 0 "#PWR017" H 10500 4350 50  0001 C CNN
 F 1 "VCC" H 10500 4650 50  0000 C CNN
 F 2 "" H 10500 4500 50  0000 C CNN
@@
 $EndComp
 $Comp
-L VCC #PWR?
+L VCC #PWR018
 U 1 1 586AE442
 P 10500 3500
-F 0 "#PWR?" H 10500 3350 50  0001 C CNN
+F 0 "#PWR018" H 10500 3350 50  0001 C CNN
 F 1 "VCC" H 10500 3650 50  0000 C CNN
 F 2 "" H 10500 3500 50  0000 C CNN
@@
 	10550 3500 10500 3500
 $Comp
-L GND #PWR?
+L GND #PWR019
 U 1 1 586AE701
 P 10500 3700
-F 0 "#PWR?" H 10500 3450 50  0001 C CNN
+F 0 "#PWR019" H 10500 3450 50  0001 C CNN
 F 1 "GND" H 10500 3550 50  0000 C CNN
 F 2 "" H 10500 3700 50  0000 C CNN
@@
 DC_C
 $Comp
-L GND #PWR?
+L GND #PWR020
 U 1 1 5871A688
 P 5850 1000
-F 0 "#PWR?" H 5850 750 50  0001 C CNN
+F 0 "#PWR020" H 5850 750 50  0001 C CNN
 F 1 "GND" V 5850 800 50  0000 C CNN
 F 2 "" H 5850 1000 50  0000 C CNN
