File: kicad/Super7Seg.sch (KiCad schematic (older format))
At the start: 36 parts, among them CON1 AVR-ISP-6, IC1 ATMEGA328P-P, IC2 74HC238, P1 CONN_01X13, P2 CONN_01X09, P3 CONN_01X13, P4 CONN_01X09, P5 UART, P6 CONN_01X02, P7 CONN_01X02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

Commit message: Fixed unsaved schematic.
Parts:
- IC2, U1: footprint (none) -> Housings_DIP:DIP-16_W7.62mm
- P5: footprint Socket_Strips:Socket_Strip_Straight_1x06 -> misc:Strip_1x06
- P6, P7: footprint Socket_Strips:Socket_Strip_Straight_1x02 -> misc:Strip_1x02
Changed lines of the file:
@@
 F 0 "P5" H 6050 1500 50  0000 C CNN
 F 1 "UART" V 6150 1150 50  0000 C CNN
-F 2 "Socket_Strips:Socket_Strip_Straight_1x06" H 6050 1150 50  0001 C CNN
+F 2 "misc:Strip_1x06" H 6050 1150 50  0001 C CNN
 F 3 "" H 6050 1150 50  0000 C CNN
 	1    6050 1150
@@
 F 0 "P6" H 6050 2000 50  0000 C CNN
 F 1 "CONN_01X02" V 6150 1850 50  0000 C CNN
-F 2 "Socket_Strips:Socket_Strip_Straight_1x02" H 6050 1850 50  0001 C CNN
+F 2 "misc:Strip_1x02" H 6050 1850 50  0001 C CNN
 F 3 "" H 6050 1850 50  0000 C CNN
 	1    6050 1850
@@
 F 0 "P7" H 6050 2550 50  0000 C CNN
 F 1 "CONN_01X02" V 6150 2400 50  0000 C CNN
-F 2 "Socket_Strips:Socket_Strip_Straight_1x02" H 6050 2400 50  0001 C CNN
+F 2 "misc:Strip_1x02" H 6050 2400 50  0001 C CNN
 F 3 "" H 6050 2400 50  0000 C CNN
 	1    6050 2400
@@
 F 0 "U1" H 12100 4150 50  0000 C CNN
 F 1 "ULN2003A" H 12100 3950 50  0000 C CNN
-F 2 "" H 12100 4050 50  0000 C CNN
+F 2 "Housings_DIP:DIP-16_W7.62mm" H 12100 4050 50  0001 C CNN
 F 3 "" H 12100 4050 50  0000 C CNN
 	1    12100 4050
@@
 F 0 "IC2" H 10800 4650 60  0000 C CNN
 F 1 "74HC238" H 10950 3350 60  0000 C CNN
-F 2 "" H 10950 4000 60  0000 C CNN
+F 2 "Housings_DIP:DIP-16_W7.62mm" H 10950 4000 60  0001 C CNN
 F 3 "" H 10950 4000 60  0000 C CNN
 	1    10950 4000
